File: mem_sub.kicad_sch (KiCad schematic)
At the start: 7 parts, among them J1 Conn_01x50_Pin

Commit message: Finish memory and start on FPGA
Parts:
- added RN3: 22, symbol Device:R_Pack08
- added RN4: 22 O, symbol Device:R_Pack04
- added RN5: 27 Ohm, symbol Device:R_Pack04
- added U13, U14, U15: 74LS158, symbol 74xx:74LS158
- added U16, U17: 74LS240, symbol 74xx:74LS240
- added U18: 74LS04, symbol 74xx:74LS04
Connections:
- net +5VD: now also U13.16 (VCC), U14.16 (VCC), U15.16 (VCC), U16.20 (VCC), U17.20 (VCC)
- net GND: now also U13.2 (I0a), U13.3 (I1a), U13.5 (I0b), U13.6 (I1b), U13.8 (GND), U14.8 (GND), U15.8 (GND), U16.10 (GND), U17.10 (GND), U17.2 (I0a), U17.4 (I1a), U17.6 (I2a), U17.8 (I3a)
- new net: RN5.7 (R2.2), U18.6
- new net: RN3.10 (R7.2), U16.16 (O1a)
- new net: RN3.11 (R6.2), U16.14 (O2a)
- new net: RN3.12 (R5.2), U16.12 (O3a)
- new net: RN3.13 (R4.2), U16.9 (O0b)
- new net: RN3.14 (R3.2), U16.7 (O1b)
- new net: RN3.15 (R2.2), U16.5 (O2b)
- new net: RN3.16 (R1.2), U16.3 (O3b)
- new net: RN3.9 (R8.2), U16.18 (O0a)
- new net: RN5.5 (R4.2), U18.2
- new net: RN5.6 (R3.2), U18.4
- new net: RN5.8 (R1.2), U18.8
- new net: RN4.8 (R1.2), U17.3 (O3b)
- new net: RN4.7 (R2.2), U17.5 (O2b)
- new net: RN4.6 (R3.2), U17.7 (O1b)
- new net: RN4.5 (R4.2), U17.9 (O0b)
- new net BMAA0: RN4.4 (R4.1)
- new net BMAA1: RN3.8 (R8.1)
- new net BMAA2: RN3.7 (R7.1)
- new net BMAA3: RN3.6 (R6.1)
- new net BMAA4: RN3.5 (R5.1)
- new net BMAA5: RN3.4 (R4.1)
- new net BMAA6: RN3.3 (R3.1)
- new net BMAA7: RN3.2 (R2.1)
- new net BMAA8: RN3.1 (R1.1)
- new net BMCAS0: U18.9
- new net BMCAS1: U18.5
- new net BMCAS2: U18.3
- new net BMCAS3: U18.1
- new net BMSWT0: RN4.2 (R2.1)
- new net MA10: U15.11 (I0d)
- new net MA11: U15.14 (I0c)
- new net MA12: U15.5 (I0b)
- new net MA13: U15.2 (I0a)
- new net MA14: U14.11 (I0d)
- new net MA15: U14.14 (I0c)
- new net MA16: U14.5 (I0b)
- new net MA17: U14.2 (I0a)
- new net MA18: U13.10 (I1d)
- new net MA19: U13.11 (I0d)
- new net MA2: U15.10 (I1d)
- new net MA20: U13.13 (I1c)
- new net MA21: U13.14 (I0c)
- new net MA3: U15.13 (I1c)
- new net MA4: U15.6 (I1b)
- new net MA5: U15.3 (I1a)
- new net MA6: U14.10 (I1d)
- new net MA7: U14.13 (I1c)
- new net MA8: U14.6 (I1b)
- new net MA9: U14.3 (I1a)
- new net MAA0: U17.11 (I0b)
- new net MAA1: U16.2 (I0a)
- new net MAA2: U16.4 (I1a)
- new net MAA3: U16.6 (I2a)
- new net MAA4: U16.8 (I3a)
- new net MAA5: U16.11 (I0b)
- new net MAA6: U16.13 (I1b)
- new net MAA7: U16.15 (I2b)
- new net MAA8: U16.17 (I3b)
- new net MSWT0: U17.15 (I2b)
- new net RAS8: U17.13 (I1b), U17.17 (I3b)
- new net RAS80: RN4.1 (R1.1)
- new net RAS81: RN4.3 (R3.1)
- new net ~{CAS0}: RN5.1 (R1.1)
- new net ~{CAS1}: RN5.2 (R2.1)
- new net ~{CAS2}: RN5.3 (R3.1)
- new net ~{CAS3}: RN5.4 (R4.1)
- new net ~{MAA0}: U15.9 (Zd)
- new net ~{MAA1}: U15.12 (Zc)
- new net ~{MAA2}: U15.7 (Zb)
- new net ~{MAA3}: U15.4 (Za)
- new net ~{MAA4}: U14.9 (Zd)
- new net ~{MAA5}: U14.12 (Zc)
- new net ~{MAA6}: U14.7 (Zb)
- new net ~{MAA7}: U14.4 (Za)
- new net ~{MAA8}: U13.9 (Zd)
- new net ~{MAA9}: U13.12 (Zc)
- new net ~{SELCOL}: U13.1 (S), U14.1 (S), U15.1 (S)
- new net ~{SG1}: U13.15 (E), U14.15 (E), U15.15 (E), U16.1 (OEa), U16.19 (OEb), U17.1 (OEa), U17.19 (OEb)
- no-connect marks 0 -> 7
